File: pihat_rs485_pwr.brd (EAGLE design)
At the start: 56 x 65 mm, 36 parts, among them J1 RASPBERRYPI-40-PIN-GPIO_PTH_N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, Q1 MOSFET-N2N7002, Q2 MOSFET-N2N7002, Q3 MOSFET-N2N7002, Q4 MOSFET-P_SMD, Q5 BIPOLAR_TRANS_ARRAY, U1 MAX481CSA

Commit message: 10/20/17, schrunk board size
Parts:
- removed POWER: TERMBLK_3PINNOSILK, UPenn:TERMBLK_3PIN_90_NOSILK
- added J3: BARREL_JACK_3PIN, UPenn:2.1_BARREL_JACK_3PIN
- added PS2: 1.0A, UPenn:R-78-EXX
- J1: value RASPBERRYPI-40-PIN-GPIO_PTH_NO_SHROUND -> RASPBERRYPI-12-PIN-GPIO_NO_SHROUD; device UPenn:2X20 -> UPenn:PI_2X6
- moved C1 47.0 mm to (74.9, 5.35)
- moved R11 47.0 mm to (58.1, 22.1)
- moved R12 47.0 mm to (58.1, 16.8)
- moved R13 47.0 mm to (58.9, 12.5)
- moved R14 47.0 mm to (58.9, 8.91)
- moved RTCB 47.0 mm to (58.9, 5.35)
- moved PWR 47.0 mm to (80.5, 28.5)
- moved R2 47.0 mm to (63.2, 5.35)
- moved R6 47.0 mm to (85.6, 28.5)
- moved R1 46.8 mm to (19.7, 14.4), flipped to the bottom, turned to 90 degrees
- moved R3 42.7 mm to (21.4, 11.1), flipped to the bottom, turned to 270 degrees
- moved Q5 42.2 mm to (27.3, 12.5), flipped to the bottom
- moved Q4 41.6 mm to (24.7, 9.46), flipped to the bottom
- moved C2 41.4 mm to (26.1, 15.9), flipped to the bottom, turned to 0 degrees
- moved TX 39.3 mm to (6.62, 1.51), turned to 180 degrees
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Connections:
- net 3.3V: no longer J1.17
- net GND: now also J3.GND, J3.GNDBRK, PS2.GND; no longer J1.14, J1.20, J1.25, J1.30, J1.34, J1.39, POWER.1, POWER.2, PS1.GND
- net N$2: now also J1.12; no longer J1.15
- net N$8: now also PS2.VOUT; no longer PS1.VOUT
- net VIN: now also J3.PWR, PS2.VIN; no longer POWER.3, PS1.VIN
Routing:
- net 3.3V: track 89.7 -> 0.00 mm, vias 3 -> 0
- net N$22: track 56.9 -> 0.00 mm, vias 1 -> 0
- net N$16: track 56.4 -> 0.00 mm
- net N$3: track 53.4 -> 4.00 mm
- net 5V: track 42.9 -> 1.82 mm
- net N$25: track 31.6 -> 0.23 mm
- net N$13: track 31.3 -> 0.12 mm
- net N$27: track 19.1 -> 1.27 mm
- net N$2: track 16.0 -> 0.00 mm
- net N$8: track 20.0 -> 5.53 mm
- net N$7: track 12.1 -> 0.00 mm
- net N$26: track 10.1 -> 0.00 mm
- net N$5: track 8.03 -> 0.00 mm
- net N$29: track 6.87 -> 0.00 mm
- net N$28: track 6.87 -> 0.00 mm
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Other:
- board size 56 x 65 mm -> 56 x 25.7 mm
