File: pihat_rs485_pwr.sch (EAGLE design)
At the start: 36 parts, among them J1 RASPBERRYPI-40-PIN-GPIO_PTH_N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, Q1 MOSFET-N2N7002, Q2 MOSFET-N2N7002, Q3 MOSFET-N2N7002, Q4 MOSFET-P_SMD, Q5 BIPOLAR_TRANS_ARRAY, U1 MAX481CSA

Commit message: 10/20/17, schrunk board size
Parts:
- removed POWER: TERMBLK_3PINNOSILK, UPenn:TERMBLK_3PINNOSILK
- added J3: BARREL_JACK_3PIN, UPenn:BARREL_JACK_3PIN
- added PS2: 1.0A, UPenn:R-78-E5.0
- J1: value RASPBERRYPI-40-PIN-GPIO_PTH_NO_SHROUND -> RASPBERRYPI-12-PIN-GPIO_NO_SHROUD; device UPenn:RASPBERRYPI-40-PIN-GPIO_PTH_NO_SHROUND -> UPenn:RASPBERRYPI-12-PIN-GPIO_NO_SHROUD
Connections:
- net GND: now also J3.GND, J3.GNDBRK, PS2.GND; no longer POWER.1, POWER.2, PS1.GND
- net N$2: now also J1.GP18#; no longer J1.GP22
- net N$8: now also PS2.5V; no longer PS1.5V
- net VIN: now also J3.PWR, PS2.VIN; no longer POWER.3, PS1.VIN
Other:
- moved on the sheet: PS1
Changed lines of the file:
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@@
 <part name="SUPPLY9" library="SparkFun-PowerSymbols" deviceset="3.3V" device=""/>
 <part name="485" library="UPenn" deviceset="TERMBLK_3PIN" device="NOSILK"/>
-<part name="POWER" library="UPenn" deviceset="TERMBLK_3PIN" device="NOSILK"/>
 <part name="S1" library="UPenn" deviceset="DPDT_DIP_SMD" device=""/>
 <part name="R15" library="SparkFun-Resistors" deviceset="RESISTOR" device="0603" value="33K"/>
@@
 <part name="SUPPLY10" library="SparkFun-PowerSymbols" deviceset="5V" device=""/>
 <part name="U$4" library="UPenn" deviceset="UPENN_SHIELD" device="_.3_SILK"/>
-<part name="J1" library="UPenn" deviceset="RASPBERRYPI-40-PIN-GPIO" device="_PTH_NO_SHROUND" value="RASPBERRYPI-40-PIN-GPIO_PTH_NO_SHROUND"/>
+<part name="J1" library="UPenn" deviceset="RASPBERRYPI-12-PIN-GPIO" device="_NO_SHROUD" value="RASPBERRYPI-12-PIN-GPIO_NO_SHROUD"/>
 <part name="Q4" library="UPenn" deviceset="MOSFET-P" device="_SMD"/>
 <part name="F1" library="UPenn" deviceset="FUSE" device=""/>
@@
 <part name="GND12" library="SparkFun-PowerSymbols" deviceset="GND" device=""/>
 <part name="PS1" library="UPenn" deviceset="D24V22F5" device=""/>
+<part name="J3" library="UPenn" deviceset="BARREL_JACK_3PIN" device=""/>
+<part name="PS2" library="UPenn" deviceset="R-78-E5.0" device="" value="1.0A"/>
 </parts>
 <sheets>
@@
 <instance part="SUPPLY9" gate="G$1" x="115.57" y="95.25" rot="R270"/>
 <instance part="485" gate="G$1" x="29.21" y="147.32" rot="MR0"/>
-<instance part="POWER" gate="G$1" x="213.36" y="128.27" rot="MR180"/>
 <instance part="S1" gate="G$1" x="85.09" y="95.25" rot="R90"/>
 <instance part="R15" gate="G$1" x="102.87" y="90.17" rot="R180"/>
@@
 <instance part="GND10" gate="1" x="218.44" y="64.77"/>
 <instance part="GND12" gate="1" x="153.67" y="71.12"/>
-<instance part="PS1" gate="G$1" x="175.26" y="121.92"/>
+<instance part="PS1" gate="G$1" x="217.17" y="105.41"/>
+<instance part="J3" gate="G$1" x="217.17" y="124.46" rot="MR0"/>
+<instance part="PS2" gate="G$1" x="175.26" y="119.38"/>
 </instances>
 <busses>
@@
 <net name="VIN" class="0">
 <segment>
-<wire x1="210.82" y1="125.73" x2="200.66" y2="125.73" width="0.1524" layer="91"/>
+<wire x1="212.09" y1="125.73" x2="200.66" y2="125.73" width="0.1524" layer="91"/>
 <pinref part="SUPPLY3" gate="G$1" pin="VIN"/>
-<pinref part="POWER" gate="G$1" pin="3"/>
+<pinref part="J3" gate="G$1" pin="PWR"/>
 </segment>
 <segment>
 <pinref part="SUPPLY2" gate="G$1" pin="VIN"/>
 <wire x1="160.02" y1="128.27" x2="165.1" y2="128.27" width="0.1524" layer="91"/>
-<pinref part="PS1" gate="G$1" pin="VIN"/>
+<wire x1="165.1" y1="121.92" x2="165.1" y2="128.27" width="0.1524" layer="91"/>
+<pinref part="PS2" gate="G$1" pin="VIN"/>
 <wire x1="167.64" y1="121.92" x2="165.1" y2="121.92" width="0.1524" layer="91"/>
-<wire x1="165.1" y1="121.92" x2="165.1" y2="128.27" width="0.1524" layer="91"/>
 </segment>
 </net>
 <net name="GND" class="0">
 <segment>
-<wire x1="210.82" y1="120.65" x2="203.2" y2="120.65" width="0.1524" layer="91"/>
+<wire x1="212.09" y1="120.65" x2="203.2" y2="120.65" width="0.1524" layer="91"/>
 <wire x1="203.2" y1="120.65" x2="200.66" y2="120.65" width="0.1524" layer="91"/>
-<wire x1="210.82" y1="123.19" x2="203.2" y2="123.19" width="0.1524" layer="91"/>
+<wire x1="212.09" y1="123.19" x2="203.2" y2="123.19" width="0.1524" layer="91"/>
 <wire x1="203.2" y1="123.19" x2="203.2" y2="120.65" width="0.1524" layer="91"/>
 <junction x="203.2" y="120.65"/>
 <pinref part="GND3" gate="1" pin="GND"/>
-<pinref part="POWER" gate="G$1" pin="2"/>
-<pinref part="POWER" gate="G$1" pin="1"/>
+<pinref part="J3" gate="G$1" pin="GNDBRK"/>
+<pinref part="J3" gate="G$1" pin="GND"/>
 </segment>
 <segment>
@@
 <pinref part="GND2" gate="1" pin="GND"/>
 <wire x1="160.02" y1="123.19" x2="162.56" y2="123.19" width="0.1524" layer="91"/>
-<pinref part="PS1" gate="G$1" pin="GND"/>
+<wire x1="162.56" y1="119.38" x2="162.56" y2="123.19" width="0.1524" layer="91"/>
+<pinref part="PS2" gate="G$1" pin="GND"/>
 <wire x1="167.64" y1="119.38" x2="162.56" y2="119.38" width="0.1524" layer="91"/>
-<wire x1="162.56" y1="119.38" x2="162.56" y2="123.19" width="0.1524" layer="91"/>
 </segment>
 <segment>
@@
 <pinref part="S1" gate="G$1" pin="4&gt;"/>
 <wire x1="82.55" y1="90.17" x2="78.74" y2="90.17" width="0.1524" layer="91"/>
-<wire x1="78.74" y1="90.17" x2="78.74" y2="48.26" width="0.1524" layer="91"/>
-<pinref part="J1" gate="G$1" pin="GP22"/>
-<wire x1="78.74" y1="48.26" x2="46.99" y2="48.26" width="0.1524" layer="91"/>
+<wire x1="78.74" y1="90.17" x2="78.74" y2="50.8" width="0.1524" layer="91"/>
+<pinref part="J1" gate="G$1" pin="GP18#"/>
+<wire x1="46.99" y1="50.8" x2="78.74" y2="50.8" width="0.1524" layer="91"/>
 </segment>
 </net>
@@
 <pinref part="Q3" gate="G$1" pin="G"/>
 <wire x1="104.14" y1="35.56" x2="109.22" y2="35.56" width="0.1524" layer="91"/>
-<wire x1="54.61" y1="76.2" x2="54.61" y2="50.8" width="0.1524" layer="91"/>
-<wire x1="54.61" y1="50.8" x2="104.14" y2="50.8" width="0.1524" layer="91"/>
-<wire x1="104.14" y1="50.8" x2="104.14" y2="35.56" width="0.1524" layer="91"/>
+<wire x1="54.61" y1="76.2" x2="54.61" y2="53.34" width="0.1524" layer="91"/>
+<wire x1="54.61" y1="53.34" x2="104.14" y2="53.34" width="0.1524" layer="91"/>
+<wire x1="104.14" y1="53.34" x2="104.14" y2="35.56" width="0.1524" layer="91"/>
 <junction x="54.61" y="76.2"/>
 <pinref part="J1" gate="G$1" pin="RXI"/>
@@
 <segment>
 <pinref part="F1" gate="G$1" pin="P$1"/>
-<wire x1="167.64" y1="116.84" x2="151.13" y2="116.84" width="0.1524" layer="91"/>
 <wire x1="151.13" y1="116.84" x2="151.13" y2="111.76" width="0.1524" layer="91"/>
-<pinref part="PS1" gate="G$1" pin="5V"/>
-</segment>
-</net>
+<pinref part="PS2" gate="G$1" pin="5V"/>
+<wire x1="151.13" y1="116.84" x2="167.64" y2="116.84" width="0.1524" layer="91"/>
+</segment>
+</net>
